File: MDM00001/MDM00001.brd (EAGLE design)
At the start: 96.5 x 61.9 mm, 54 parts, among them J1 POWER_JACKPTH, Q1 FDN340P, U1 ATMEGA328P_PDIP, U10 SN74HC02DR, U3 CD4011BM, U4 NCP1117ST50T3G, U5 DRV8837DSGR, U6 DRV8837DSGR, U9 FT232RLSSOP

Commit message: Updated README and added PDF Files
Other:
- board text added: "Designed by: B. Carrizales"
Changed lines of the file:
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@@
 <wire x1="96.5" y1="61.9" x2="0" y2="61.9" width="0" layer="20"/>
 <wire x1="0" y1="61.9" x2="0" y2="0" width="0" layer="20"/>
+<text x="77.47" y="3.81" size="1.778" layer="16" rot="MR0">Designed by: B. Carrizales</text>
 </plain>
 <attributes>
