File: MDM00001/MDM00001.sch (EAGLE design)
At the start: 74 parts, among them J1 POWER_JACKPTH, Q1 FDN340P, U1 ATMEGA328P_PDIP, U3 TPS73633DBVR, U4 NCP1117ST50T3G, U5 DRV8837DSGR, U6 DRV8837DSGR, U7 DRV8837DSGR, U8 DRV8837DSGR, U9 FT232RLSSOP

Commit message: Finished Major Layout
Finished major layout and updated schematic. Regenerated BOM.
Parts:
- removed C14, C15, C16, C17: 0.1uF, SparkFun-Passives:CAP0603-CAP
- removed C6: 0.01uF, SparkFun-Passives:CAP0603-CAP
- removed C9: 1.0uF, SparkFun-Passives:CAP0603-CAP
- removed CR10, CR11, CR12, CR13, CR14, CR15, CR16, CR9: SMD26PL, DiscreteActive:SMD26PL
- removed JP5: 2-TERMINAL, Connectors:2-TERMINAL
- removed JP6, JP7: (no value), SparkFun-Connectors:M081X08
- removed JP8: (no value), SparkFun-Connectors:M06SIP
- removed JP9: M102MM, SparkFun-Connectors:M102MM
- removed R1: 1M, SparkFun-Passives:RESISTOR0603-RES
- removed U7, U8: DRV8837DSGR, PowerICs:DRV8837DSGR
- added C5: 0.1uF, SparkFun-Passives:CAP0603-CAP
- added U10: SN74HC02DR, LogicICs:SN74HC02DR
- JP4: value 2-TERMINAL -> (none); device Connectors:2-TERMINAL -> SparkFun-Connectors:M05PTH
- U3: value TPS73633DBVR -> CD4011BM; device regulators:TPS73633DBVR -> LogicICs:CD4011BM
Connections:
- removed net !SLEEP3: U7.!SLEEP
- removed net !SLEEP4: U8.!SLEEP
- removed net IN1C: U7.IN1
- removed net IN1D: U8.IN1
- removed net IN2C: U7.IN2
- removed net IN2D: U8.IN2
- removed net N$11: C6.1, U3.NR
- removed net N$14: C16.1, U8.VCC
- removed net N$16: C14.1, U7.VCC
- removed net N$18: C12.1, U6.VCC
- removed net N$21: C10.1, U5.VCC
- removed net OUT1C: CR10.1, JP4.2, U7.OUT1
- removed net OUT1D: CR13.1, CR15.2, JP5.2, U8.OUT1
- removed net OUT2C: CR11.1, CR12.2, JP4.1, U7.OUT2
- removed net OUT2D: CR14.1, CR16.2, JP5.1, U8.OUT2
- removed net PB0: JP9.1, U1.PB0(ICP)
- removed net PD3: JP6.4, U1.PD3(INT1)
- removed net PD4: JP6.5, U1.PD4(XCK/T0)
- removed net PD5: JP6.6, U1.PD5(T1)
- removed net PD6: JP6.7, U1.PD6(AIN0)
- removed net PD7: JP6.8, U1.PD7(AIN1)
- removed net RXD: JP6.1
- removed net TXD: JP6.2
- new net DIR1: U1.PD4(XCK/T0), U10A.I1, U3A.I0, U3A.I1
- new net DIR2: U1.PD7(AIN1), U10C.I1, U3B.I0, U3B.I1
- new net N$27: U10B.I1, U3A.O1
- new net N$3: U10D.I1, U3B.O1
- new net PWM1: U1.PD3(INT1), U10A.I0, U10B.I0
- new net PWM2: U1.PD6(AIN0), U10C.I0, U10D.I0
- net !SLEEP1: now also U1.PD5(T1)
- net !SLEEP2: now also U1.PB0(ICP)
- net 3.3V: no longer JP7.4, U3.OUT
- net 5V: now also C10.1, C12.1, JP4.1, U10A.14, U3A.14, U3C.I0, U3C.I1, U3D.I0, U3D.I1, U5.VCC, U6.VCC; no longer C9.1, JP7.2, JP7.5, U3.IN
- net AD0: now also JP4.2; no longer JP8.1
- net AD1: now also JP4.3; no longer JP8.2
- net AD2: now also JP4.4; no longer JP8.3
- net AD3: no longer JP8.4
- net AD4/SDA: no longer JP8.5, JP9.9
- net AD5/SCL: no longer JP8.6, JP9.10
- net AREF: no longer JP9.8
- net DTR: now also C5.1
- net GND: now also JP4.5, U10A.7, U3A.7; no longer C14.2, C15.2, C16.2, C17.2, C6.2, C9.2, CR12.1, CR15.1, CR16.1, CR9.1, JP7.6, JP7.7, JP9.7, U3.GND, U7.GND, U8.GND
- net IN1A: now also U10A.O1
- net IN1B: now also U10C.O1
- net IN2A: now also U10B.O1
- net IN2B: now also U10D.O1
- net MISO: no longer JP9.5
- net MOSI: no longer JP9.4
- net N$1: no longer R1.2
- net N$2: no longer R1.1
- net PB1: no longer JP9.2
- net PD2: no longer JP6.3
- net RESET: now also C5.2; no longer JP7.3
- net SCK: no longer JP9.6
- net SS: no longer JP9.3
- net VIN: no longer C15.1, C17.1, CR10.2, CR11.2, CR13.2, CR14.2, JP7.8, U7.VM, U8.VM
Other:
- note added: "0"
- note added: "1 of 2"
- note added: "2 of 2"
- note added: "4 CH DC Motor Driver Microcontroller Board"
- moved on the sheet: C10, C11, C12, C13, C7, C8, CR1, CR2, CR3, CR4, CR5, CR6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

Commit message: Updated README and added PDF Files
Other:
- note added: "2 CH DC Motor Driver Microcontroller Board"
- note added: "Designed by: B. Carrizales"
- note removed: "4 CH DC Motor Driver Microcontroller Board"
Changed lines of the file:
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@@
 <sheet>
 <plain>
-<text x="119.38" y="-81.28" size="2.54" layer="91">4 CH DC Motor Driver
+<text x="119.38" y="-81.28" size="2.54" layer="91">2 CH DC Motor Driver
 Microcontroller Board</text>
 <text x="177.546" y="-82.55" size="1.778" layer="91">1 of 2</text>
 <text x="177.292" y="-75.438" size="1.778" layer="91">0</text>
+<text x="71.12" y="-81.28" size="1.778" layer="91">Designed by: B. Carrizales</text>
 </plain>
 <instances>
@@
 <sheet>
 <plain>
-<text x="96.52" y="-48.26" size="2.54" layer="91">4 CH DC Motor Driver
+<text x="96.52" y="-48.26" size="2.54" layer="91">2 CH DC Motor Driver
 Microcontroller Board</text>
 <text x="152.4" y="-50.8" size="1.778" layer="91">2 of 2</text>
 <text x="152.4" y="-43.18" size="1.778" layer="91">0</text>
+<text x="45.72" y="-45.72" size="1.778" layer="91">Designed by: B. Carrizales</text>
 </plain>
 <instances>
